File: kicad-global/RP2040-VCO.kicad_sch (KiCad schematic)
At the start: 58 parts, among them J1 Out, J2 Conn_01x06_Female, J3 Conn_01x06_Male, J4 Conn_01x08_Female, J5 Conn_01x08_Male, J6 V/oct, J7 Inv CV, J8 Power Input, SW1 SW_MEC_LOW_PROF_LED, SW2 SW_SPDT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

Commit message: v1.5
reverse pots following issue raised on github
Connections:
- net +3V3: now also CHORD1.3, TUNE1.3; no longer CHORD1.1, TUNE1.1
- net +5V: now also INV1.3; no longer INV1.1
- net GND: now also CHORD1.1, INV1.1, TUNE1.1; no longer CHORD1.3, INV1.3, TUNE1.3
Changed lines of the file:
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@@
 (kicad_sch
-	(version 20231120)
+	(version 20250114)
 	(generator "eeschema")
-	(generator_version "8.0")
+	(generator_version "9.0")
 	(paper "A4")
 	(title_block
 		(title "RP2040 VCO")
-		(date "2025-04-15")
-		(rev "1.4")
+		(date "2025-10-29")
+		(rev "1.5")
 		(company "Bleep Sound")
 	)
+	(text "replace output with a DAC ?\nSee DAC8164ICPW for example.\nWould force a code modification\nhttps://deepbluembedded.com/digital-to-analog-converter-dac-waveform-generation-with-mcu/"
+		(exclude_from_sim no)
+		(at 170.434 29.21 0)
+		(effects
+			(font
+				(size 1.27 1.27)
+			)
+		)
+	)
+	(text "RP2040 chord style VCO by Hagiwo\nSMD version by BleepSound"
+		(exclude_from_sim no)
+		(at 121.92 22.86 0)
+		(effects
+			(font
+				(size 1.8 1.8)
+			)
+			(justify left bottom)
+		)
+	)
 	(junction
 		(at 123.19 175.26)
@@
 		)
 	)
-	(text "replace output with a DAC ?\nSee DAC8164ICPW for example.\nWould force a code modification\nhttps://deepbluembedded.com/digital-to-analog-converter-dac-waveform-generation-with-mcu/"
-		(exclude_from_sim no)
-		(at 170.434 29.21 0)
-		(effects
-			(font
-				(size 1.27 1.27)
-			)
-		)
-	)
-	(text "RP2040 chord style VCO by Hagiwo\nSMD version by BleepSound"
-		(exclude_from_sim no)
-		(at 121.92 22.86 0)
-		(effects
-			(font
-				(size 1.8 1.8)
-			)
-			(justify left bottom)
-		)
-	)
 	(label "TunePot"
 		(at 29.21 59.69 90)
-		(fields_autoplaced yes)
 		(effects
 			(font
@@
 	(label "Push_SW"
 		(at 224.79 81.28 180)
-		(fields_autoplaced yes)
 		(effects
 			(font
@@
 	(label "Push_SW"
 		(at 86.36 54.61 0)
-		(fields_autoplaced yes)
 		(effects
 			(font
@@
 	(label "Tune"
 		(at 57.15 59.69 180)
-		(fields_autoplaced yes)
 		(effects
 			(font
@@
 	(label "Chord"
 		(at 57.15 85.09 180)
-		(fields_autoplaced yes)
 		(effects
 			(font
@@
 	(label "InvJack"
 		(at 278.13 100.33 180)
-		(fields_autoplaced yes)
 		(effects
 			(font
@@
 	(label "SW_0"
 		(at 278.13 107.95 180)
-		(fields_autoplaced yes)
 		(effects
 			(font
@@
 	(label "SW_1"
 		(at 278.13 113.03 180)
-		(fields_autoplaced yes)
 		(effects
 			(font
@@
 	(label "InvPot"
 		(at 243.84 80.01 0)
-		(fields_autoplaced yes)
 		(effects
 			(font
@@
 	(label "ChordPot"
 		(at 29.21 85.09 90)
-		(fields_autoplaced yes)
 		(effects
 			(font
@@
 	(label "V{slash}oct"
 		(at 88.9 44.45 0)
-		(fields_autoplaced yes)
 		(effects
 			(font
@@
 	(label "InvJack"
 		(at 113.03 138.43 270)
-		(fields_autoplaced yes)
 		(effects
 			(font
@@
 	(label "V{slash}octJack"
 		(at 241.3 102.87 0)
-		(fields_autoplaced yes)
 		(effects
 			(font
@@
 	(label "InvPot"
 		(at 275.59 80.01 180)
-		(fields_autoplaced yes)
 		(effects
 			(font
@@
 	(label "OutJack"
 		(at 259.08 46.99 270)
-		(fields_autoplaced yes)
 		(effects
 			(font
@@
 	(label "SW_0"
 		(at 88.9 59.69 0)
-		(fields_autoplaced yes)
 		(effects
 			(font
@@
 	(label "V{slash}octJack"
 		(at 278.13 102.87 180)
-		(fields_autoplaced yes)
 		(effects
 			(font
@@
 	(label "V{slash}oct"
 		(at 72.39 114.3 180)
-		(fields_autoplaced yes)
 		(effects
 			(font
@@
 	(label "Inv"
 		(at 88.9 49.53 0)
-		(fields_autoplaced yes)
 		(effects
 			(font
@@
 	(label "TunePot"
 		(at 243.84 82.55 0)
-		(fields_autoplaced yes)
 		(effects
 			(font
@@
 	(label "SW_0"
 		(at 241.3 107.95 0)
-		(fields_autoplaced yes)
 		(effects
 			(font
@@
 	(label "Chord"
 		(at 88.9 52.07 0)
-		(fields_autoplaced yes)
 		(effects
 			(font
@@
 	(label "ChordPot"
 		(at 275.59 85.09 180)
-		(fields_autoplaced yes)
 		(effects
 			(font
@@
 	(label "InvPot"
 		(at 106.68 113.03 90)
-		(fields_autoplaced yes)
 		(effects
 			(font
@@
 	(label "InvJack"
 		(at 241.3 100.33 0)
-		(fields_autoplaced yes)
 		(effects
 			(font
@@
 	(label "OutJack"
 		(at 241.3 97.79 0)
-		(fields_autoplaced yes)
 		(effects
 			(font
@@
 	(label "SW_1"
 		(at 124.46 44.45 180)
-		(fields_autoplaced yes)
 		(effects
 			(font
@@
 	(label "V{slash}octJack"
 		(at 31.75 114.3 270)
-		(fields_autoplaced yes)
 		(effects
 			(font
@@
 	(label "SW_1"
 		(at 241.3 113.03 0)
-		(fields_autoplaced yes)
 		(effects
 			(font
@@
 	(label "ChordPot"
 		(at 243.84 85.09 0)
-		(fields_autoplaced yes)
 		(effects
 			(font
@@
 	(label "SW_1"
 		(at 207.01 109.22 180)
-		(fields_autoplaced yes)
 		(effects
 			(font
@@
 	(label "Out"
 		(at 173.99 44.45 0)
-		(fields_autoplaced yes)
 		(effects
 			(font
@@
 	(label "Push_SW"
 		(at 241.3 110.49 0)
-		(fields_autoplaced yes)
 		(effects
 			(font
@@
 	(label "Inv"
 		(at 232.41 143.51 180)
-		(fields_autoplaced yes)
 		(effects
 			(font
@@
 	(label "SW_0"
 		(at 207.01 104.14 180)
-		(fields_autoplaced yes)
 		(effects
 			(font
@@
 	(label "Out"
 		(at 124.46 46.99 180)
-		(fields_autoplaced yes)
 		(effects
 			(font
@@
 	(label "Push_SW"
 		(at 278.13 110.49 180)
-		(fields_autoplaced yes)
 		(effects
 			(font
@@
 	(label "Tune"
 		(at 88.9 46.99 0)
-		(fields_autoplaced yes)
 		(effects
 			(font
@@
 	(label "TunePot"
 		(at 275.59 82.55 180)
-		(fields_autoplaced yes)
 		(effects
 			(font
@@
 	(label "OutJack"
 		(at 278.13 97.79 180)
-		(fields_autoplaced yes)
 		(effects
 			(font
@@
 		(lib_id "Device:R_POT")
 		(at 22.86 59.69 0)
+		(mirror x)
 		(unit 1)
 		(exclude_from_sim no)
@@
 		(dnp no)
 		(property "Reference" "TUNE1"
-			(at 21.59 60.96 0)
+			(at 21.59 58.42 0)
 			(effects
 				(font
@@
 		)
 		(property "Value" "10k"
-			(at 21.59 58.42 0)
+			(at 21.59 60.96 0)
 			(effects
 				(font
@@
 		(lib_id "Device:R_POT")
 		(at 22.86 85.09 0)
+		(mirror x)
 		(unit 1)
 		(exclude_from_sim no)
@@
 		(dnp no)
 		(property "Reference" "CHORD1"
-			(at 21.59 86.36 0)
+			(at 21.59 83.82 0)
 			(effects
 				(font
@@
 		)
 		(property "Value" "10k"
-			(at 21.59 83.82 0)
+			(at 21.59 86.36 0)
 			(effects
 				(font
@@
 		(lib_id "Device:R_POT")
 		(at 100.33 113.03 0)
+		(mirror x)
 		(unit 1)
 		(exclude_from_sim no)
@@
 		(dnp no)
 		(property "Reference" "INV1"
-			(at 99.06 114.3 0)
+			(at 99.06 111.76 0)
 			(effects
 				(font
@@
 		)
 		(property "Value" "10k"
-			(at 99.06 111.76 0)
+			(at 99.06 114.3 0)
 			(effects
 				(font
@@
 		)
 	)
+	(embedded_fonts no)
 )
